Commit message: Reached a good urdf robo-car model

File: catkin_ws/src/ros_car_description/urdf/ros_car.xacro (robot description, xacro)
@@ -15,4 +15,17 @@
     <color rgba="0.5 0.5 0.5 1.0"/>
   </material>
+  <!-- Dummy Link for Root Inertia -->
+  <link name="base_dummy">
+    <inertial>
+      <mass value="0.01"/>
+      <inertia ixx="0.00001" ixy="0.0" ixz="0.0"
+               iyy="0.00001" iyz="0.0" izz="0.00001"/>
+    </inertial>
+  </link>
+  <joint name="base_dummy_joint" type="fixed">
+    <parent link="base_dummy"/>
+    <child link="base_link"/>
+    <origin xyz="0 0 0" rpy="0 0 0"/>
+  </joint>
   <!-- Main Loom -->
   <link name="base_link">
@@ -30,8 +43,9 @@
     <inertial>
       <mass value="2.0"/>
-      <inertia ixx="0.1" iyy="0.1" izz="0.1"/>
+      <inertia ixx="0.1" ixy="0.0" ixz="0.0"
+               iyy="0.1" iyz="0.0" izz="0.1"/>
     </inertial>
   </link>
-  <!-- Lefr Wheel -->
+  <!-- Left Wheel -->
   <link name="wheel_left">
     <visual>
@@ -40,5 +54,5 @@
       </geometry>
       <material name="black"/>
-      <origin rpy="0 0 ${pi/2}"/>
+      <origin rpy="${pi/2} 0 0"/>
     </visual>
     <collision>
@@ -46,16 +60,18 @@
         <cylinder radius="${wheel_radius}" length="${wheel_width}"/>
       </geometry>
+      <origin rpy="${pi/2} 0 0"/>
     </collision>
     <inertial>
       <mass value="0.1"/>
-      <inertia ixx="0.001" iyy="0.001" izz="0.001"/>
+      <inertia ixx="0.001" ixy="0.0" ixz="0.0"
+              iyy="0.001" iyz="0.0" izz="0.001"/>
     </inertial>
   </link>
-  <joint name="joint_wheel_left" type="continuous">
-    <parent link="base_link"/>
-    <child link="wheel_left"/>
-    <origin xyz="0 ${wheel_separation/2} 0" rpy="0 0 0"/>
-    <axis xyz="0 1 0"/>
-  </joint>
+<joint name="joint_wheel_left" type="continuous">
+  <parent link="base_link"/>
+  <child link="wheel_left"/>
+  <origin xyz="${base_length/4} ${wheel_separation/3} -${chassis_height/2}" rpy="0 0 0"/>
+  <axis xyz="0 1 0"/>
+</joint>
   <!-- Right Wheel -->
   <link name="wheel_right">
@@ -65,5 +81,5 @@
       </geometry>
       <material name="black"/>
-      <origin rpy="0 0 ${pi/2}"/>
+      <origin rpy="${pi/2} 0 0"/>
     </visual>
     <collision>
@@ -71,8 +87,10 @@
         <cylinder radius="${wheel_radius}" length="${wheel_width}"/>
       </geometry>
+      <origin rpy="${pi/2} 0 0"/>
     </collision>
     <inertial>
       <mass value="0.1"/>
-      <inertia ixx="0.001" iyy="0.001" izz="0.001"/>
+      <inertia ixx="0.001" ixy="0.0" ixz="0.0"
+              iyy="0.001" iyz="0.0" izz="0.001"/>
     </inertial>
   </link>
@@ -80,5 +98,5 @@
     <parent link="base_link"/>
     <child link="wheel_right"/>
-    <origin xyz="0 -${wheel_separation/2} 0" rpy="0 0 0"/>
+    <origin xyz="${base_length/4} -${wheel_separation/3} -${chassis_height/2}" rpy="0 0 0"/>
     <axis xyz="0 1 0"/>
   </joint>
@@ -98,5 +116,6 @@
     <inertial>
       <mass value="0.05"/>
-      <inertia ixx="0.0001" iyy="0.0001" izz="0.0001"/>
+      <inertia ixx="0.0001" ixy="0.0" ixz="0.0"
+               iyy="0.0001" iyz="0.0" izz="0.0001"/>
     </inertial>
   </link>
@@ -107,24 +126,24 @@
   </joint>
   <!-- Plugins -->
-<gazebo>
-  <plugin name="diff_drive_controller" filename="libgazebo_ros_diff_drive.so">
-    <ros>
-      <namespace>/</namespace>
-      <remapping>cmd_vel:=/cmd_vel</remapping>
-      <remapping>odom:=/odom</remapping>
-    </ros>
-    <commandTimeout>1.0</commandTimeout>
-    <wheelSeparation>${wheel_separation}</wheelSeparation>
-    <wheelDiameter>${2 * wheel_radius}</wheelDiameter>
-    <wheelAcceleration>0.0</wheelAcceleration>
-    <wheelTorque>5.0</wheelTorque>
-    <updateRate>50.0</updateRate>
-    <leftJoint>joint_wheel_left</leftJoint>
-    <rightJoint>joint_wheel_right</rightJoint>
-    <publishOdom>true</publishOdom>
-    <odomFrame>odom</odomFrame>
-    <odomTopic>odom</odomTopic>
-    <robotBaseFrame>base_link</robotBaseFrame>
-  </plugin>
-</gazebo>
+  <gazebo>
+    <plugin name="diff_drive_controller" filename="libgazebo_ros_diff_drive.so">
+      <ros>
+        <namespace>/</namespace>
+        <remapping>cmd_vel:=/cmd_vel</remapping>
+        <remapping>odom:=/odom</remapping>
+      </ros>
+      <commandTimeout>1.0</commandTimeout>
+      <wheelSeparation>${wheel_separation}</wheelSeparation>
+      <wheelDiameter>${2 * wheel_radius}</wheelDiameter>
+      <wheelAcceleration>0.0</wheelAcceleration>
+      <wheelTorque>5.0</wheelTorque>
+      <updateRate>50.0</updateRate>
+      <leftJoint>joint_wheel_left</leftJoint>
+      <rightJoint>joint_wheel_right</rightJoint>
+      <publishOdom>true</publishOdom>
+      <odomFrame>odom</odomFrame>
+      <odomTopic>odom</odomTopic>
+      <robotBaseFrame>base_link</robotBaseFrame>
+    </plugin>
+  </gazebo>
 </robot>

Commit message: A lot of things, but autonomus system works well

File: catkin_ws/src/ros_car_description/urdf/ros_car.xacro (robot description, xacro)
@@ -15,17 +15,4 @@
     <color rgba="0.5 0.5 0.5 1.0"/>
   </material>
-  <!-- Dummy Link for Root Inertia -->
-  <link name="base_dummy">
-    <inertial>
-      <mass value="0.01"/>
-      <inertia ixx="0.00001" ixy="0.0" ixz="0.0"
-               iyy="0.00001" iyz="0.0" izz="0.00001"/>
-    </inertial>
-  </link>
-  <joint name="base_dummy_joint" type="fixed">
-    <parent link="base_dummy"/>
-    <child link="base_link"/>
-    <origin xyz="0 0 0" rpy="0 0 0"/>
-  </joint>
   <!-- Main Loom -->
   <link name="base_link">

Commit message: Waypoints service on, now the autonomus system work very well. Added secret key (private param), deleted useless nodes, some refactoring, added doc-strings

File: catkin_ws/src/ros_car_description/urdf/ros_car.xacro (robot description, xacro)
@@ -2,10 +2,10 @@
 <robot name="ros_car" xmlns:xacro="http://ros.org/wiki/xacro">
   <!-- Local Params -->
+  <xacro:property name="chassis_height" value="0.05"/>
+  <xacro:property name="base_length" value="0.4"/>
+  <xacro:property name="base_width" value="0.2"/>
   <xacro:property name="wheel_radius" value="0.05"/>
   <xacro:property name="wheel_width" value="0.02"/>
   <xacro:property name="wheel_separation" value="0.3"/>
-  <xacro:property name="base_length" value="0.4"/>
-  <xacro:property name="base_width" value="0.2"/>
-  <xacro:property name="chassis_height" value="0.05"/>
   <!-- Materials -->
   <material name="black">
@@ -114,23 +114,29 @@
   <!-- Plugins -->
   <gazebo>
-    <plugin name="diff_drive_controller" filename="libgazebo_ros_diff_drive.so">
-      <ros>
-        <namespace>/</namespace>
-        <remapping>cmd_vel:=/cmd_vel</remapping>
-        <remapping>odom:=/odom</remapping>
-      </ros>
-      <commandTimeout>1.0</commandTimeout>
-      <wheelSeparation>${wheel_separation}</wheelSeparation>
-      <wheelDiameter>${2 * wheel_radius}</wheelDiameter>
-      <wheelAcceleration>0.0</wheelAcceleration>
-      <wheelTorque>5.0</wheelTorque>
-      <updateRate>50.0</updateRate>
-      <leftJoint>joint_wheel_left</leftJoint>
-      <rightJoint>joint_wheel_right</rightJoint>
-      <publishOdom>true</publishOdom>
-      <odomFrame>odom</odomFrame>
-      <odomTopic>odom</odomTopic>
-      <robotBaseFrame>base_link</robotBaseFrame>
-    </plugin>
+      <plugin name="diff_drive_controller" filename="libgazebo_ros_diff_drive.so">
+          <ros>
+              <namespace>/</namespace>
+              <remapping>odom:=/odom</remapping>
+              <remapping>cmd_vel:=/cmd_vel</remapping>
+          </ros>
+          <publishOdom>true</publishOdom>
+          <publishTf>true</publishTf>
+          <publishOdomTF>true</publishOdomTF>
+          <publishWheelTF>false</publishWheelTF>
+          <commandTimeout>1.0</commandTimeout>
+          <updateRate>50.0</updateRate>
+          <wheelTorque>5.0</wheelTorque>
+          <wheelAcceleration>0.0</wheelAcceleration>
+          <wheelDiameter>${2 * wheel_radius}</wheelDiameter>
+          <wheelSeparation>${wheel_separation}</wheelSeparation>
+          <robotBaseFrame>base_link</robotBaseFrame>
+          <odometryFrame>odom</odometryFrame>
+          <odometryTopic>odom</odometryTopic>
+          <commandTopic>cmd_vel</commandTopic>
+          <publishWheelJointState>true</publishWheelJointState>
+          <leftJoint>joint_wheel_left</leftJoint>
+          <rightJoint>joint_wheel_right</rightJoint>
+          <rosDebugLevel>INFO</rosDebugLevel>
+      </plugin>
   </gazebo>
 </robot>

Commit message: Added a first laser scan implementation, to do an bug/wall-follow strategy or move_base strategy

File: catkin_ws/src/ros_car_description/urdf/ros_car.xacro (robot description, xacro)
@@ -34,4 +34,28 @@
     </inertial>
   </link>
+  <!-- Scanner -->
+  <link name="laser_link">
+    <visual>
+      <geometry>
+        <box size="0.05 0.05 0.05"/>
+      </geometry>
+      <material name="black"/>
+    </visual>
+    <collision>
+      <geometry>
+        <box size="0.05 0.05 0.05"/>
+      </geometry>
+    </collision>
+    <inertial>
+      <mass value="0.05"/>
+      <inertia ixx="0.0001" ixy="0.0" ixz="0.0"
+               iyy="0.0001" iyz="0.0" izz="0.0001"/>
+    </inertial>
+  </link>
+  <joint name="joint_laser_link" type="fixed">
+    <parent link="base_link"/>
+    <child link="laser_link"/>
+    <origin xyz="0.2 0 0.05" rpy="0 0 0"/>
+  </joint>
   <!-- Left Wheel -->
   <link name="wheel_left">
@@ -55,10 +79,10 @@
     </inertial>
   </link>
-<joint name="joint_wheel_left" type="continuous">
-  <parent link="base_link"/>
-  <child link="wheel_left"/>
-  <origin xyz="${base_length/4} ${wheel_separation/3} -${chassis_height/2}" rpy="0 0 0"/>
-  <axis xyz="0 1 0"/>
-</joint>
+  <joint name="joint_wheel_left" type="continuous">
+    <parent link="base_link"/>
+    <child link="wheel_left"/>
+    <origin xyz="${base_length/4} ${wheel_separation/3} -${chassis_height/2}" rpy="0 0 0"/>
+    <axis xyz="0 1 0"/>
+  </joint>
   <!-- Right Wheel -->
   <link name="wheel_right">
@@ -113,30 +137,63 @@
   </joint>
   <!-- Plugins -->
+  <gazebo reference="laser_link">						    <!-- Attach sensor to 'laser_link' -->
+    <sensor type="ray" name="laser_sensor">
+      <alwaysOn>true</alwaysOn>						      <!-- Keep sensor active -->
+      <update_rate>20</update_rate>					    <!-- Publish at 20 Hz -->
+      <visualize>true</visualize>						    <!-- Show beams in Gazebo -->
+      <topicName>scan</topicName>						    <!-- ROS topic for LaserScan -->
+      <pose>0 0 0 0 0 0</pose>						      <!-- Sensor pose relative to link -->
+      <ray>
+        <scan>
+          <horizontal>
+            <samples>360</samples>					    <!-- Number of beams -->
+            <resolution>1</resolution>				  <!-- Subdivisions between beams -->
+            <min_angle>-1.5708</min_angle>			<!-- -90 degrees in radians -->
+            <max_angle>1.5708</max_angle>				<!-- +90 degrees in radians -->
+          </horizontal>
+        </scan>
+        <range>
+          <min>0.12</min>						            <!-- Minimum detect distance (m) -->
+          <max>2.0</max>						            <!-- Maximum detect distance (m) -->
+          <resolution>0.01</resolution>				  <!-- Range resolution (m) -->
+        </range>
+        <noise>
+          <type>gaussian</type>					        <!-- Noise model type -->
+          <mean>0.0</mean>						          <!-- Mean of noise -->
+          <stddev>0.01</stddev>					        <!-- Standard deviation of noise -->
+        </noise>
+      </ray>
+      <plugin name="gazebo_ros_laser_controller" filename="libgazebo_ros_laser.so">
+        <topicName>scan</topicName>					    <!-- Same ROS topic name -->
+        <frameName>laser_link</frameName>				<!-- Laser data frame -->
+      </plugin>
+    </sensor>
+  </gazebo>
   <gazebo>
-      <plugin name="diff_drive_controller" filename="libgazebo_ros_diff_drive.so">
-          <ros>
-              <namespace>/</namespace>
-              <remapping>odom:=/odom</remapping>
-              <remapping>cmd_vel:=/cmd_vel</remapping>
-          </ros>
-          <publishOdom>true</publishOdom>
-          <publishTf>true</publishTf>
-          <publishOdomTF>true</publishOdomTF>
-          <publishWheelTF>false</publishWheelTF>
-          <commandTimeout>1.0</commandTimeout>
-          <updateRate>50.0</updateRate>
-          <wheelTorque>5.0</wheelTorque>
-          <wheelAcceleration>0.0</wheelAcceleration>
-          <wheelDiameter>${2 * wheel_radius}</wheelDiameter>
-          <wheelSeparation>${wheel_separation}</wheelSeparation>
-          <robotBaseFrame>base_link</robotBaseFrame>
-          <odometryFrame>odom</odometryFrame>
-          <odometryTopic>odom</odometryTopic>
-          <commandTopic>cmd_vel</commandTopic>
-          <publishWheelJointState>true</publishWheelJointState>
-          <leftJoint>joint_wheel_left</leftJoint>
-          <rightJoint>joint_wheel_right</rightJoint>
-          <rosDebugLevel>INFO</rosDebugLevel>
-      </plugin>
+    <plugin name="diff_drive_controller" filename="libgazebo_ros_diff_drive.so">
+      <ros>
+        <namespace>/</namespace>					                      <!-- ROS namespace -->
+        <remapping>odom:=/odom</remapping>				              <!-- Remap /odom topic -->
+        <remapping>cmd_vel:=/cmd_vel</remapping>			          <!-- Remap /cmd_vel topic -->
+      </ros>
+      <publishOdom>true</publishOdom>					                  <!-- Publish odometry messages -->
+      <publishTf>true</publishTf>						                    <!-- Publish TF transforms -->
+      <publishOdomTF>true</publishOdomTF>				                <!-- Publish odom->base_link TF -->
+      <publishWheelTF>false</publishWheelTF>				            <!-- No wheel TF broadcast -->
+      <commandTimeout>1.0</commandTimeout>				              <!-- Stop if no cmd_vel after 1s -->
+      <updateRate>50.0</updateRate>					                    <!-- Plugin update frequency (Hz) -->
+      <wheelTorque>5.0</wheelTorque>					                  <!-- Max torque on wheels -->
+      <wheelAcceleration>0.0</wheelAcceleration>				        <!-- Max wheel acceleration (0=unlimited) -->
+      <wheelDiameter>${2 * wheel_radius}</wheelDiameter>			  <!-- Wheel diameter (m) -->
+      <wheelSeparation>${wheel_separation}</wheelSeparation>		<!-- Distance between wheels (m) -->
+      <robotBaseFrame>base_link</robotBaseFrame>				        <!-- Robot's main reference frame -->
+      <odometryFrame>odom</odometryFrame>					              <!-- Frame for odom data -->
+      <odometryTopic>odom</odometryTopic>					              <!-- Topic for odom data -->
+      <commandTopic>cmd_vel</commandTopic>					            <!-- Topic for velocity cmds -->
+      <publishWheelJointState>true</publishWheelJointState>			<!-- Publish wheel joint states -->
+      <leftJoint>joint_wheel_left</leftJoint>				            <!-- Name of the left joint -->
+      <rightJoint>joint_wheel_right</rightJoint>				        <!-- Name of the right joint -->
+      <rosDebugLevel>INFO</rosDebugLevel>					              <!-- Debug level -->
+    </plugin>
   </gazebo>
 </robot>

Commit message: Added a full wall-following logic for the autonomus car, some correction and params tuning, added a lot of params, deleted the useless files

File: catkin_ws/src/ros_car_description/urdf/ros_car.xacro (robot description, xacro)
@@ -83,4 +83,5 @@
     <child link="wheel_left"/>
     <origin xyz="${base_length/4} ${wheel_separation/3} -${chassis_height/2}" rpy="0 0 0"/>
+    <dynamics damping="0.1" friction="0.1"/>
     <axis xyz="0 1 0"/>
   </joint>
@@ -110,4 +111,5 @@
     <child link="wheel_right"/>
     <origin xyz="${base_length/4} -${wheel_separation/3} -${chassis_height/2}" rpy="0 0 0"/>
+    <dynamics damping="0.1" friction="0.1"/>
     <axis xyz="0 1 0"/>
   </joint>
@@ -149,6 +151,6 @@
             <samples>360</samples>					    <!-- Number of beams -->
             <resolution>1</resolution>				  <!-- Subdivisions between beams -->
-            <min_angle>-3.1416</min_angle>      <!-- -180 gradi in radianti -->
-            <max_angle>3.1416</max_angle>       <!-- +180 gradi in radianti -->
+            <min_angle>-3.1416</min_angle>      <!-- -180° rads -->
+            <max_angle>3.1416</max_angle>       <!-- +180° rads -->
           </horizontal>
         </scan>
@@ -182,5 +184,5 @@
       <publishWheelTF>false</publishWheelTF>				            <!-- No wheel TF broadcast -->
       <commandTimeout>1.0</commandTimeout>				              <!-- Stop if no cmd_vel after 1s -->
-      <updateRate>50.0</updateRate>					                    <!-- Plugin update frequency (Hz) -->
+      <updateRate>100</updateRate>					                    <!-- Plugin update frequency (Hz) -->
       <wheelTorque>5.0</wheelTorque>					                  <!-- Max torque on wheels -->
       <wheelAcceleration>0.0</wheelAcceleration>				        <!-- Max wheel acceleration (0=unlimited) -->
